File: PushbuttonPowerPathControllerWithSupervisor_LTC2952.kicad_sch (KiCad schematic)
At the start: 20 parts, among them J1 PJ-082BH, J2 Raspberry_Pi_2_3, Q1 DMP3036SSD-13, SW1 SW_Push, U1 D36V28F5, U2 LTC2952CF-PBF

Commit message: 回路図コメント追記
Parts:
- added R9: 10k, Resistor_SMD:R_0603_1608Metric, symbol Device:R_Small
Connections:
- net +3V3: now also R9.1
- net INT: now also J2.37 (GPIO26), R9.2; no longer J2.22 (GPIO25), R7.2
- net KILL: now also R7.2; no longer J2.37 (GPIO26)
- net G1STAT: now reaches D3.2 (A), R1.2
- net G1STAT: now also J2.22 (GPIO25)
Other:
- note added: "12V/(551k+100k) =18uA"
- note added: "Threshold is 0.5V"
- note added: "tKILL,ONBLANK is 400ms"
- moved on the sheet: BT1, C1, C2, D1, D2, D3, J1, J2, Q1A, Q1B, R1, R2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
